Commit message: improve mashes for meshcat

File: urdf/icub_description/urdf/icub.urdf (robot description, URDF)
Before this commit: robot iCub, 56 links, 55 joints
Links:
- link chest: geometry collision mesh filename=package://icub_description/meshes/upmc/collision/icub_simpl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 scale=1 1 1; visual mesh filename=package://icub_description/meshes/upmc/visual/icub_chest.obj scale=1 1 1
- link head: geometry collision mesh filename=package://icub_description/meshes/upmc/collision/icub_simpl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 scale=1 1 1; visual mesh filename=package://icub_description/meshes/upmc/visual/icub_head.obj scale=1 1 1
- link l_foot: geometry collision mesh filename=package://icub_description/meshes/upmc/collision/icub_simpl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 scale=1 1 1; visual mesh filename=package://icub_description/meshes/upmc/visual/icub_l_foot.o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 scale=1 1 1
- link l_hand: geometry collision mesh filename=package://icub_description/meshes/upmc/collision/icub_simpl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 scale=1 1 1; visual mesh filename=package://icub_description/meshes/upmc/visual/icub_l_hand.o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 scale=1 1 1
- link l_upper_arm: geometry collision mesh filename=package://icub_description/meshes/upmc/collision/icub_simpl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 scale=1 1 1; visual mesh filename=package://icub_description/meshes/upmc/visual/icub_l_arm.obj scale=1 1 1
- link neck_1: geometry collision mesh filename=package://icub_description/meshes/upmc/collision/icub_simpl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 scale=1 1 1; visual mesh filename=package://icub_description/meshes/upmc/visual/icub_neck_1.o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 scale=1 1 1
- link neck_2: geometry collision mesh filename=package://icub_description/meshes/upmc/collision/icub_simpl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 scale=1 1 1; visual mesh filename=package://icub_description/meshes/upmc/visual/icub_neck_2.o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 scale=1 1 1
- link r_foot: geometry collision mesh filename=package://icub_description/meshes/upmc/collision/icub_simpl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 scale=1 1 1; visual mesh filename=package://icub_description/meshes/upmc/visual/icub_r_foot.o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 scale=1 1 1
- link r_hand: geometry collision mesh filename=package://icub_description/meshes/upmc/collision/icub_simpl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 scale=1 1 1; visual mesh filename=package://icub_description/meshes/upmc/visual/icub_r_hand.o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 scale=1 1 1
- link r_upper_arm: geometry collision mesh filename=package://icub_description/meshes/upmc/collision/icub_simpl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 scale=1 1 1; visual mesh filename=package://icub_description/meshes/upmc/visual/icub_r_arm.obj scale=1 1 1
